Commit message: created basic urdf with documentation of what everything does

File: src/spex_rover_description/src/description/spex_rover_description.urdf (robot description, URDF)
Before this commit: robot spex_rover, 0 links, 0 joints
Links:
- added link base_footprint
- added link base_link; visual box size=${base_length} ${base_width} ${base_height}
Joints:
- added joint base_joint: type fixed, parent base_link, child base_footprint, origin xyz=0.0 0.0 ${-(wheel_radius+wheel_zoff)} rpy=0 0 0

Commit message: updated front and back wheel config

File: src/spex_rover_description/src/description/spex_rover_description.urdf (robot description, URDF)
Before this commit: robot spex_rover, 2 links, 1 joints
Joints:
- joint base_joint: origin xyz=0.0 0.0 ${-(wheel_radius+wheel_zoff)} rpy=0 0 0 -> xyz=0.0 0.0 ${-(wheel_radius+wheel_front_zoff)} rpy=0 0 0

Commit message: I made a (temporary) urdf for the rover, consisting of a box with wheels and joints

File: src/spex_rover_description/src/description/spex_rover_description.urdf (robot description, URDF)
Before this commit: robot spex_rover, 2 links, 1 joints
Links:
- added link drivewhl_bl_link, mass 0.5; collision cylinder length=0.04 radius=0.1; visual cylinder length=0.04 radius=0.1
- added link drivewhl_br_link, mass 0.5; collision cylinder length=0.04 radius=0.1; visual cylinder length=0.04 radius=0.1
- added link drivewhl_fl_link, mass 0.5; collision cylinder length=0.04 radius=0.1; visual cylinder length=0.04 radius=0.1
- added link drivewhl_fr_link, mass 0.5; collision cylinder length=0.04 radius=0.1; visual cylinder length=0.04 radius=0.1
- added link imu_link, mass 0.1; collision box size=0.1 0.1 0.1; visual box size=0.1 0.1 0.1
- link base_link: mass None -> 40; geometry collision box size=0.75 0.75 0.6; visual box size=0.75 0.75 0.6
Joints:
- added joint drivewhl_bl_joint: type continuous, parent base_link, child drivewhl_bl_link, origin xyz=-0.25 0.4 -0.3 rpy=0 0 0, axis 0 1 0
- added joint drivewhl_br_joint: type continuous, parent base_link, child drivewhl_br_link, origin xyz=-0.25 -0.4 -0.3 rpy=0 0 0, axis 0 1 0
- added joint drivewhl_fl_joint: type continuous, parent base_link, child drivewhl_fl_link, origin xyz=0.25 0.4 -0.3 rpy=0 0 0, axis 0 1 0
- added joint drivewhl_fr_joint: type continuous, parent base_link, child drivewhl_fr_link, origin xyz=0.25 -0.4 -0.3 rpy=0 0 0, axis 0 1 0
- added joint imu_joint: type fixed, parent base_link, child imu_link, origin xyz=0 0 0.01
- joint base_joint: origin xyz=0.0 0.0 ${-(wheel_radius+wheel_front_zoff)} rpy=0 0 0 -> xyz=0.0 0.0 -0.4 rpy=0 0 0
